File: _autosave-pwm_driver.kicad_pcb (KiCad board)
At the start: 2 copper layers, 56.6 x 57.7 mm, 41 parts, among them J1 V_{In}, J2 GND_{In}, J3 SolderPad, J4 SolderPad, Q1 BC817, Q2 BC807, Q3 BUK7880-55A, U1 TLV2372, U2 LM393

Commit message: photo added from working device
Parts:
- Q3: value BUK7880-55A -> TSM900N06CW_RPG; footprint Package_TO_SOT_SMD:SOT-223-3_TabPin2 -> TRANS_TSM900N06CW_RPG:TRANS_TSM900N06CW_RPG
- R1, R2: value 100k -> 51k
Changed lines of the file:
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@@
       (effects (font (size 1 1) (thickness 0.15)))
     )
-    (fp_text value "100k" (at 0 1.82 90) (layer "F.Fab")
+    (fp_text value "51k" (at 0 1.82 90) (layer "F.Fab")
       (effects (font (size 1 1) (thickness 0.15)))
     )
@@
       (effects (font (size 1 1) (thickness 0.15)))
     )
-    (fp_text value "100k" (at 0 1.82 90) (layer "F.Fab")
+    (fp_text value "51k" (at 0 1.82 90) (layer "F.Fab")
       (effects (font (size 1 1) (thickness 0.15)))
     )
@@
     )
   )
-  (footprint "Package_TO_SOT_SMD:SOT-223-3_TabPin2" (layer "F.Cu")
-    (at 108.41 134.29)
-    (descr "module CMS SOT223 4 pins")
-    (tags "CMS SOT")
-    (property "Sheetfile" "pwm_driver.kicad_sch")
-    (property "Sheetname" "")
-    (attr smd)
-    (fp_text reference "Q3" (at 0 -4.5) (layer "F.SilkS")
-      (effects (font (size 1 1) (thickness 0.15)))
-    )
-    (fp_text value "BUK7880-55A" (at 0 4.5) (layer "F.Fab")
-      (effects (font (size 1 1) (thickness 0.15)))
-    )
-    (fp_text user "${REFERENCE}" (at 0 0 90) (layer "F.Fab")
-      (effects (font (size 0.8 0.8) (thickness 0.12)))
-    )
-    (fp_line (start 1.91 -3.41) (end 1.91 -2.15) (layer "F.SilkS") (width 0.12))
-    (fp_line (start -1.85 3.41) (end 1.91 3.41) (layer "F.SilkS") (width 0.12))
-    (fp_line (start -4.1 -3.41) (end 1.91 -3.41) (layer "F.SilkS") (width 0.12))
-    (fp_line (start 1.91 3.41) (end 1.91 2.15) (layer "F.SilkS") (width 0.12))
-    (fp_line (start -4.4 3.6) (end 4.4 3.6) (layer "F.CrtYd") (width 0.05))
-    (fp_line (start -4.4 -3.6) (end -4.4 3.6) (layer "F.CrtYd") (width 0.05))
-    (fp_line (start 4.4 -3.6) (end -4.4 -3.6) (layer "F.CrtYd") (width 0.05))
-    (fp_line (start 4.4 3.6) (end 4.4 -3.6) (layer "F.CrtYd") (width 0.05))
-    (fp_line (start -1.85 -2.35) (end -1.85 3.35) (layer "F.Fab") (width 0.1))
-    (fp_line (start 1.85 -3.35) (end 1.85 3.35) (layer "F.Fab") (width 0.1))
-    (fp_line (start -0.85 -3.35) (end 1.85 -3.35) (layer "F.Fab") (width 0.1))
-    (fp_line (start -1.85 -2.35) (end -0.85 -3.35) (layer "F.Fab") (width 0.1))
-    (fp_line (start -1.85 3.35) (end 1.85 3.35) (layer "F.Fab") (width 0.1))
-    (pad "1" smd rect (at -3.15 -2.3) (size 2 1.5) (layers "F.Cu" "F.Paste" "F.Mask")
-      (net 1 "/U_{FET_driver}") (pinfunction "G") (pintype "input"))
-    (pad "2" smd rect (at -3.15 0) (size 2 1.5) (layers "F.Cu" "F.Paste" "F.Mask")
-      (net 11 "/FET_Drain") (pinfunction "D") (pintype "passive"))
-    (pad "2" smd rect (at 3.15 0) (size 2 3.8) (layers "F.Cu" "F.Paste" "F.Mask")
-      (net 11 "/FET_Drain") (pinfunction "D") (pintype "passive"))
-    (pad "3" smd rect (at -3.15 2.3) (size 2 1.5) (layers "F.Cu" "F.Paste" "F.Mask")
-      (net 6 "GND") (pinfunction "S") (pintype "passive"))
-    (model "${KICAD6_3DMODEL_DIR}/Package_TO_SOT_SMD.3dshapes/SOT-223.wrl"
-      (offset (xyz 0 0 0))
-      (scale (xyz 1 1 1))
-      (rotate (xyz 0 0 0))
-    )
-  )
   (footprint "Capacitor_SMD:C_1206_3216Metric_Pad1.33x1.80mm_HandSolder" (layer "F.Cu")
     (at 96.98 92.126 180)
@@
       (net 2 "/U_{PWM}") (pinfunction "1") (pintype "passive"))
   )
+  (footprint "TRANS_TSM900N06CW_RPG:TRANS_TSM900N06CW_RPG" (layer "F.Cu")
+    (at 108.375 134.3)
+    (property "MANUFACTURER" "Taiwan Semiconductor")
+    (property "MAXIMUM_PACKAGE_HEIGHT" "1.80mm")
+    (property "PARTREV" "D1706")
+    (property "STANDARD" "Manufacturer recommendation")
+    (property "Sheetfile" "pwm_driver.kicad_sch")
+    (property "Sheetname" "")
+    (attr through_hole)
+    (fp_text reference "Q3" (at -1.08 -5.135) (layer "F.SilkS")
+      (effects (font (size 1 1) (thickness 0.15)))
+    )
+    (fp_text value "TSM900N06CW_RPG" (at 9.08 5.135) (layer "F.Fab")
+      (effects (font (size 1 1) (thickness 0.15)))
+    )
+    (fp_line (start 1.75 3.25) (end -1.75 3.25) (layer "F.SilkS") (width 0.127))
+    (fp_line (start -1.75 3.25) (end -1.75 -3.25) (layer "F.SilkS") (width 0.127))
+    (fp_line (start -1.75 -3.25) (end 1.75 -3.25) (layer "F.SilkS") (width 0.127))
+    (fp_line (start 1.75 -3.25) (end 1.75 3.25) (layer "F.SilkS") (width 0.127))
+    (fp_circle (center -5.005 -2.3) (end -4.905 -2.3) (layer "F.SilkS") (width 0.2) (fill none))
+    (fp_line (start 4.25 3.5) (end 4.25 -3.5) (layer "F.CrtYd") (width 0.05))
+    (fp_line (start -4.25 -3.5) (end -4.25 3.5) (layer "F.CrtYd") (width 0.05))
+    (fp_line (start -4.25 3.5) (end 4.25 3.5) (layer "F.CrtYd") (width 0.05))
+    (fp_line (start 4.25 -3.5) (end -4.25 -3.5) (layer "F.CrtYd") (width 0.05))
+    (fp_line (start 1.75 -3.25) (end 1.75 3.25) (layer "F.Fab") (width 0.127))
+    (fp_line (start -1.75 -3.25) (end 1.75 -3.25) (layer "F.Fab") (width 0.127))
+    (fp_line (start -1.75 3.25) (end -1.75 -3.25) (layer "F.Fab") (width 0.127))
+    (fp_line (start 1.75 3.25) (end -1.75 3.25) (layer "F.Fab") (width 0.127))
+    (fp_circle (center -5.005 -2.3) (end -4.905 -2.3) (layer "F.Fab") (width 0.2) (fill none))
+    (pad "1" smd rect locked (at -3.2 -2.3) (size 1.6 1.2) (layers "F.Cu" "F.Paste" "F.Mask")
+      (net 1 "/U_{FET_driver}") (pintype "passive"))
+    (pad "2" smd rect locked (at -3.2 0) (size 1.6 1.2) (layers "F.Cu" "F.Paste" "F.Mask")
+      (net 11 "/FET_Drain") (pintype "passive"))
+    (pad "3" smd rect locked (at -3.2 2.3) (size 1.6 1.2) (layers "F.Cu" "F.Paste" "F.Mask")
+      (net 6 "GND") (pintype "passive"))
+    (pad "4" smd rect locked (at 3.2 0) (size 1.6 3.3) (layers "F.Cu" "F.Paste" "F.Mask")
+      (net 11 "/FET_Drain") (pintype "passive"))
+  )
   (footprint "Resistor_SMD:R_1206_3216Metric_Pad1.30x1.75mm_HandSolder" (layer "F.Cu")
