File: pwm_driver.kicad_pcb (KiCad board)
At the start: 2 copper layers, 56.6 x 57.7 mm, 41 parts, among them J1 V_{In}, J2 GND_{In}, J3 SolderPad, J4 SolderPad, Q1 BC817, Q2 BC807, Q3 TSM900N06CW_RPG, U1 TLV2372, U2 LM393

Commit message: some more GND vias added
Routing:
- net GND: vias 162 -> 217
